File: PCB - CPU V1/CPU & Memory.kicad_sch (KiCad schematic)
At the start: 29 parts, among them U1 74HCT132, U10 ATF22V10C, U11 ATF22V10C, U12 SST39SF010, U13 74HCT32, U5 AS6C4008, U6 AS6C4008, U7 AS6C4008, U8 AS6C4008

Commit message: CPU Card
Parts:
- gave numbers to parts that had none: 19
