File: PCB - CPU V1/PCB - CPU V1.kicad_sch (KiCad schematic)
At the start: 25 parts, among them J2 +5V DC, SW1 POWER, SW2 RESET, U2 74HCT14, U3 74HCT74, U4 74HCT112, X1 16MHz

Commit message: CPU Card
Parts:
- gave numbers to parts that had none: 1
